File: EUISOpcb.kicad_pcb (KiCad board)
At the start: 2 copper layers, 281.1 x 76.2 mm, 121 parts, among them P1 USB_C_Plug_USB2.0, SW1 SW_Push, U1 ATmega32U4-AU, Y1 16MHz

Commit message: Completed PCB
Completed the PCB by adding 7u Support and new decorations
Parts:
- added MX53: MX-NoLED, MX_Only:MXOnly-7U-ReversedStabilizers-NoLED, F.Cu at (173.9, 121.5)
- added MX54: MX-NoLED, MX_Only:MXOnly-1.25U-NoLED, F.Cu at (71.5, 121.5)
- added MX55: MX-NoLED, MX_Only:MXOnly-1.25U-NoLED, F.Cu at (95.2, 121.5)
- added MX56: MX-NoLED, MX_Only:MXOnly-1.25U-NoLED, F.Cu at (252.4, 121.5)
- added MX57: MX-NoLED, MX_Only:MXOnly-1.25U-NoLED, F.Cu at (276.2, 121.5)
- moved D46 15.5 mm to (156.8, 121.5)
- moved D50 12.3 mm to (240.5, 112.1), turned to 0 degrees
- moved D42 7.27 mm to (94.1, 114.7), turned to 180 degrees
- moved D41 2.92 mm to (80.0, 121.7)
- moved R1 0.74 mm to (11.9, 66.4)
Routing:
- net COL7: track 206.7 -> 233.1 mm
- net ROW3: track 295.9 -> 318.9 mm
- net Net-(D46-Pad2): track 6.93 -> 21.0 mm
- net COL12: track 312.6 -> 324.1 mm, vias 1 -> 5
- net COL3: track 140.9 -> 152.3 mm, vias 1 -> 3
- net Net-(D51-Pad2): track 6.70 -> 14.1 mm
- net COL13: track 332.7 -> 338.5 mm
- net GND: track 150.9 -> 147.2 mm
- net Net-(D41-Pad2): track 6.93 -> 9.73 mm
- net COL11: track 293.0 -> 295.4 mm, vias 1 -> 3
- net Net-(D52-Pad2): track 7.06 -> 9.47 mm
- net COL2: track 116.1 -> 118.5 mm
- net COL0: track 52.6 -> 55.0 mm
- net Net-(D42-Pad2): track 6.62 -> 8.88 mm
- net Net-(P1-PadA5): track 7.10 -> 9.24 mm
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- added copper zone on B.Cu, net GND
- added copper zone on F.Cu, net GND
Other:
- board text added: "LETS GET ISOLATED"
- board text added: "Sample Text"
- board text added: "Yea, we have a fucking 7 unit spacebar on this! Why? Fuck you that's why!"
