File: EUISOpcb.kicad_pcb (KiCad board)
At the start: 2 copper layers, 281.1 x 76.2 mm, 127 parts, among them P1 USB_C_Plug_USB2.0, SW1 SW_Push, U1 ATmega32U4-AU, Y1 16MHz

Commit message: Idk what I did this time
But it was definitely something, it is complete though
Parts:
- removed P1: USB_C_Plug_USB2.0, Connector_USB:USB_C_Receptacle_Amphenol_12401548E4-2A
- added G***: LOGO, cheems:FHoleSignature, F.Cu at (260.4, 79.1)
- added J1: USB_C_Receptacle_USB2.0, Connector_USB:USB_C_Receptacle_HRO_TYPE-C-31-M-12, B.Cu at (18.8, 57.5)
- R3, R4: value 22 -> 22 Ohm
- moved G*** 114.3 mm to (56.4, 107.1)
Routing:
- net +5V: track 83.7 -> 113.3 mm, vias 4 -> 8
- net Net-(J1-PadS1): track 0.00 -> 18.1 mm
- net GND: track 147.2 -> 158.1 mm, vias 4 -> 2
- net Net-(J1-PadA6): track 56.1 -> 62.7 mm, vias 0 -> 2
- net Net-(J1-PadA7): track 46.5 -> 51.6 mm
- net Net-(F1-Pad2): track 13.3 -> 17.5 mm, vias 2 -> 3
- net Net-(J1-PadA5): track 9.24 -> 12.5 mm
- net COL10: track 274.8 -> 273.6 mm
- net Net-(J1-PadB5): vias 0 -> 2
Other:
- board text added: "Floof's Got It Handled ;)"

Commit message: Complete
finished with gerbers
Parts:
- removed MX29: MX-NoLED, MX_Only:MXOnly-1U-NoLED
- added G***: LOGO, cheems:EUFlag, F.Cu at (107.5, 84.3)
- added G***: LOGO, cheems:kermit, F.Cu at (173.6, 71.6)
- added G***: LOGO, cheems:Logo, B.Cu at (232.1, 91.8)
- added G***: LOGO, cheems:Logo, B.Cu at (193.8, 92.6)
- added G***: LOGO, cheems:Logo, B.Cu at (109.4, 92.4)
- added G***: LOGO, cheems:Logo, B.Cu at (71.9, 93.3)
- added REF**: 1U, MX_Only:MXOnly-1U-NoLED, F.Cu at (69.1, 102.5)
Other:
- board text added: "All my friends in Voice Gang and IRL and finally the 40% Discord for giving me a channel"
- board text added: "Credits: Creater/PCB Design: TuckTuckFloof OG Case Design: evangs (aka THE TRASH MAN) Case Editor/Vendor/3dPrinting God: Jake from P3Dstore Amazing Silk: MeatSmoothies"
- board text added: "Hi Mom"
- board text added: "LETS GET ISO-LATED"
- board text added: "What do teens like?!? is it memes? Memes about skeletons? Piss? Communism?"
