File: _autosave-EUISOpcb.kicad_pcb (KiCad board)
At the start: 2 copper layers, 281.1 x 76.2 mm, 127 parts, among them P1 USB_C_Plug_USB2.0, SW1 SW_Push, U1 ATmega32U4-AU, Y1 16MHz

Commit message: Cheems
Cheems
Parts:
- moved G*** 114.3 mm to (56.4, 107.1)
Changed lines of the file:
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@@
   )
   (module cheems:cheems (layer F.Cu)
-    (at 170.18 96.266)
+    (at 56.388 107.061)
     (fp_text reference G*** (at 0 0) (layer F.SilkS) hide
       (effects (font (size 1.524 1.524) (thickness 0.3)))
